Commit message: Modifications matching 69359bf895516fc252d8335fcffd38e4a6553e50

File: kinova_description/urdf/j2n4s300.xacro (robot description, xacro)
@@ -52,6 +52,6 @@
     <xacro:property name="joint_2_origin_xyz" value="0 0.0016 -0.11875" />
     <xacro:property name="joint_2_origin_rpy" value="${-J_PI/2} 0 ${J_PI}" />
-    <xacro:property name="joint_2_lower_limit" value="${30/180*J_PI}" />
-    <xacro:property name="joint_2_upper_limit" value="${330/180*J_PI}" />
+    <xacro:property name="joint_2_lower_limit" value="${47/180*J_PI}" />
+    <xacro:property name="joint_2_upper_limit" value="${313/180*J_PI}" />
     <xacro:property name="joint_3" value="joint_3" />
     <xacro:property name="joint_3_type" value="revolute" />
@@ -59,6 +59,6 @@
     <xacro:property name="joint_3_origin_xyz" value="0 -0.410 0" />
     <xacro:property name="joint_3_origin_rpy" value="0 ${J_PI} 0" />
-    <xacro:property name="joint_3_lower_limit" value="${30/180*J_PI}" />
-    <xacro:property name="joint_3_upper_limit" value="${330/180*J_PI}" />
+    <xacro:property name="joint_3_lower_limit" value="${19/180*J_PI}" />
+    <xacro:property name="joint_3_upper_limit" value="${341/180*J_PI}" />
     <xacro:property name="joint_4" value="joint_4" />
     <xacro:property name="joint_4_type" value="continuous" />

File: kinova_description/urdf/j2n6s200.xacro (robot description, xacro)
@@ -56,6 +56,6 @@
     <xacro:property name="joint_2_origin_xyz" value="0 0.0016 -0.11875" />
     <xacro:property name="joint_2_origin_rpy" value="-${J_PI/2} 0 ${J_PI}" />
-    <xacro:property name="joint_2_lower_limit" value="${30/180*J_PI}" />
-    <xacro:property name="joint_2_upper_limit" value="${330/180*J_PI}" />
+    <xacro:property name="joint_2_lower_limit" value="${47/180*J_PI}" />
+    <xacro:property name="joint_2_upper_limit" value="${313/180*J_PI}" />
     <xacro:property name="joint_3" value="joint_3" />
     <xacro:property name="joint_3_type" value="revolute" />
@@ -63,6 +63,6 @@
     <xacro:property name="joint_3_origin_xyz" value="0 -0.410 0" />
     <xacro:property name="joint_3_origin_rpy" value="0 ${J_PI} 0" />
-    <xacro:property name="joint_3_lower_limit" value="${30/180*J_PI}" />
-    <xacro:property name="joint_3_upper_limit" value="${330/180*J_PI}" />
+    <xacro:property name="joint_3_lower_limit" value="${19/180*J_PI}" />
+    <xacro:property name="joint_3_upper_limit" value="${341/180*J_PI}" />
     <xacro:property name="joint_4" value="joint_4" />
     <xacro:property name="joint_4_type" value="continuous" />

File: kinova_description/urdf/j2n6s300.xacro (robot description, xacro)
@@ -56,6 +56,6 @@
     <xacro:property name="joint_2_origin_xyz" value="0 0.0016 -0.11875" />
     <xacro:property name="joint_2_origin_rpy" value="-${J_PI/2} 0 ${J_PI}" />
-    <xacro:property name="joint_2_lower_limit" value="${30/180*J_PI}" />
-    <xacro:property name="joint_2_upper_limit" value="${330/180*J_PI}" />
+    <xacro:property name="joint_2_lower_limit" value="${47/180*J_PI}" />
+    <xacro:property name="joint_2_upper_limit" value="${313/180*J_PI}" />
     <xacro:property name="joint_3" value="joint_3" />
     <xacro:property name="joint_3_type" value="revolute" />
@@ -63,6 +63,6 @@
     <xacro:property name="joint_3_origin_xyz" value="0 -0.410 0" />
     <xacro:property name="joint_3_origin_rpy" value="0 ${J_PI} 0" />
-    <xacro:property name="joint_3_lower_limit" value="${30/180*J_PI}" />
-    <xacro:property name="joint_3_upper_limit" value="${330/180*J_PI}" />
+    <xacro:property name="joint_3_lower_limit" value="${19/180*J_PI}" />
+    <xacro:property name="joint_3_upper_limit" value="${341/180*J_PI}" />
     <xacro:property name="joint_4" value="joint_4" />
     <xacro:property name="joint_4_type" value="continuous" />

File: kinova_description/urdf/j2s6s300.xacro (robot description, xacro)
@@ -56,6 +56,6 @@
     <xacro:property name="joint_2_origin_xyz" value="0 0.0016 -0.11875" />
     <xacro:property name="joint_2_origin_rpy" value="${-J_PI/2} 0 ${J_PI}"/>
-    <xacro:property name="joint_2_lower_limit" value="${30/180*J_PI}" />
-    <xacro:property name="joint_2_upper_limit" value="${330/180*J_PI}" />
+    <xacro:property name="joint_2_lower_limit" value="${47/180*J_PI}" />
+    <xacro:property name="joint_2_upper_limit" value="${313/180*J_PI}" />
     <xacro:property name="joint_3" value="joint_3" />
     <xacro:property name="joint_3_type" value="revolute" />
@@ -63,6 +63,6 @@
     <xacro:property name="joint_3_origin_xyz" value="0 -0.410 0" />
     <xacro:property name="joint_3_origin_rpy" value="0 ${J_PI} 0" />
-    <xacro:property name="joint_3_lower_limit" value="${30/180*J_PI}" />
-    <xacro:property name="joint_3_upper_limit" value="${330/180*J_PI}" />
+    <xacro:property name="joint_3_lower_limit" value="${19/180*J_PI}" />
+    <xacro:property name="joint_3_upper_limit" value="${341/180*J_PI}" />
     <xacro:property name="joint_4" value="joint_4" />
     <xacro:property name="joint_4_type" value="continuous" />

File: kinova_description/urdf/j2s7s300.xacro (robot description, xacro)
@@ -58,6 +58,6 @@
     <xacro:property name="joint_2_origin_xyz" value="0 0.0016 -0.11875" />
     <xacro:property name="joint_2_origin_rpy" value="-${J_PI/2} 0 ${J_PI}" />
-    <xacro:property name="joint_2_lower_limit" value="${30/180*J_PI}" />
-    <xacro:property name="joint_2_upper_limit" value="${330/180*J_PI}" />
+    <xacro:property name="joint_2_lower_limit" value="${47/180*J_PI}" />
+    <xacro:property name="joint_2_upper_limit" value="${313/180*J_PI}" />
     <xacro:property name="joint_3" value="joint_3" />
     <xacro:property name="joint_3_type" value="continuous" />
@@ -86,6 +86,6 @@
     <xacro:property name="joint_6_origin_xyz" value="0 0 -0.10375" />
     <xacro:property name="joint_6_origin_rpy" value="${J_PI/2} 0 ${J_PI}" />
-    <xacro:property name="joint_6_lower_limit" value="${30/180*J_PI}" />
-    <xacro:property name="joint_6_upper_limit" value="${330/180*J_PI}" />
+    <xacro:property name="joint_6_lower_limit" value="${65/180*J_PI}" />
+    <xacro:property name="joint_6_upper_limit" value="${295/180*J_PI}" />
     <xacro:property name="joint_7" value="joint_7" />
     <xacro:property name="joint_7_type" value="continuous" />

File: kinova_description/urdf/m1n4s200.xacro (robot description, xacro)
@@ -52,6 +52,6 @@
     <xacro:property name="joint_2_origin_xyz" value="0 0.0016 -0.11875" />
     <xacro:property name="joint_2_origin_rpy" value="${-J_PI/2} 0 ${J_PI}" />
-    <xacro:property name="joint_2_lower_limit" value="${30/180*J_PI}" />
-    <xacro:property name="joint_2_upper_limit" value="${330/180*J_PI}" />
+    <xacro:property name="joint_2_lower_limit" value="${50/180*J_PI}" />
+    <xacro:property name="joint_2_upper_limit" value="${310/180*J_PI}" />
     <xacro:property name="joint_3" value="joint_3" />
     <xacro:property name="joint_3_type" value="revolute" />
@@ -59,6 +59,6 @@
     <xacro:property name="joint_3_origin_xyz" value="0 -0.290 0" />
     <xacro:property name="joint_3_origin_rpy" value="0 ${J_PI} 0" />
-    <xacro:property name="joint_3_lower_limit" value="${30/180*J_PI}" />
-    <xacro:property name="joint_3_upper_limit" value="${330/180*J_PI}" />
+    <xacro:property name="joint_3_lower_limit" value="${35/180*J_PI}" />
+    <xacro:property name="joint_3_upper_limit" value="${325/180*J_PI}" />
     <xacro:property name="joint_4" value="joint_4" />
     <xacro:property name="joint_4_type" value="continuous" />

File: kinova_description/urdf/m1n6s200.xacro (robot description, xacro)
@@ -56,6 +56,6 @@
     <xacro:property name="joint_2_origin_xyz" value="0 0.0016 -0.11875" />
     <xacro:property name="joint_2_origin_rpy" value="${-J_PI/2} 0 ${J_PI}" />
-    <xacro:property name="joint_2_lower_limit" value="${30/180*J_PI}" />
-    <xacro:property name="joint_2_upper_limit" value="${330/180*J_PI}" />
+    <xacro:property name="joint_2_lower_limit" value="${50/180*J_PI}" />
+    <xacro:property name="joint_2_upper_limit" value="${310/180*J_PI}" />
     <xacro:property name="joint_3" value="joint_3" />
     <xacro:property name="joint_3_type" value="revolute" />
@@ -63,6 +63,6 @@
     <xacro:property name="joint_3_origin_xyz" value="0 -0.290 0" />
     <xacro:property name="joint_3_origin_rpy" value="0 ${J_PI} 0" />
-    <xacro:property name="joint_3_lower_limit" value="${30/180*J_PI}" />
-    <xacro:property name="joint_3_upper_limit" value="${330/180*J_PI}" />
+    <xacro:property name="joint_3_lower_limit" value="${35/180*J_PI}" />
+    <xacro:property name="joint_3_upper_limit" value="${325/180*J_PI}" />
     <xacro:property name="joint_4" value="joint_4" />
     <xacro:property name="joint_4_type" value="continuous" />

File: kinova_description/urdf/m1n6s300.xacro (robot description, xacro)
@@ -56,6 +56,6 @@
     <xacro:property name="joint_2_origin_xyz" value="0 0.0016 -0.11875" />
     <xacro:property name="joint_2_origin_rpy" value="${-J_PI/2} 0 ${J_PI}" />
-    <xacro:property name="joint_2_lower_limit" value="${30/180*J_PI}" />
-    <xacro:property name="joint_2_upper_limit" value="${330/180*J_PI}" />
+    <xacro:property name="joint_2_lower_limit" value="${50/180*J_PI}" />
+    <xacro:property name="joint_2_upper_limit" value="${310/180*J_PI}" />
     <xacro:property name="joint_3" value="joint_3" />
     <xacro:property name="joint_3_type" value="revolute" />
@@ -63,6 +63,6 @@
     <xacro:property name="joint_3_origin_xyz" value="0 -0.290 0" />
     <xacro:property name="joint_3_origin_rpy" value="0 ${J_PI} 0" />
-    <xacro:property name="joint_3_lower_limit" value="${30/180*J_PI}" />
-    <xacro:property name="joint_3_upper_limit" value="${330/180*J_PI}" />
+    <xacro:property name="joint_3_lower_limit" value="${35/180*J_PI}" />
+    <xacro:property name="joint_3_upper_limit" value="${325/180*J_PI}" />
     <xacro:property name="joint_4" value="joint_4" />
     <xacro:property name="joint_4_type" value="continuous" />
